File: ESP32ScoringDevice_PCB_THT_Rev1.2.kicad_pcb (KiCad board)
At the start: 2 copper layers, 66 x 53.3 mm, 32 parts, among them J1 Fencers Fencers, J2 Matrix + WS2812B LED Matrix, J3 timer display + MAX7219 Timer Display, J4 HC-06 module HC-06 BT module, J5 ICSP ICSP, J6 Conn_01x02, J7 Conn_01x02, J8 Buzzer Buzzer, J9 5V ext. 5V ext. Power, Q1 BC337, Q2 BC337, Q3 FQP27P06, U1 ESP32_DevKit_V1_DOIT 30pin

Commit message: Rev 1.2b
Small tweaks
Other:
- board text added: "ESP32 fencing scoring device / weapons tester github.com/pietwauters/esp32_scoring_device_hardware ©Piet Wauters 2024 GNU GPL V3.0 PCB Rev. 1.2b"
- board text added: "Fencing 3 weapons █ scoring device █ tester PCB Rev. 1.2b"
- board text removed: "ESP32 fencing scoring device / weapons tester github.com/pietwauters/esp32_scoring_device_hardware ©Piet Wauters 2024 GNU GPL V3.0 PCB Rev. 1.2"
- board text removed: "Fencing 3 weapons █ scoring device █ tester PCB Rev. 1.2"
Changed lines of the file:
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@@
 			)
 		)
-		(fp_text user "Boot"
-			(at 7.62 39.68 0)
-			(layer "F.SilkS")
-			(effects
-				(font
-					(size 1 1)
-					(thickness 0.15)
-				)
-			)
-		)
-		(fp_text user "Enable"
-			(at -7.62 39.68 0)
-			(layer "F.SilkS")
-			(effects
-				(font
-					(size 1 1)
-					(thickness 0.15)
-				)
-			)
-		)
 		(pad "1" thru_hole rect
 			(at -12.7 0)
@@
 		(layer "Edge.Cuts")
 	)
-	(gr_text "ESP32 fencing scoring device / weapons tester\ngithub.com/pietwauters/esp32_scoring_device_hardware\n©Piet Wauters 2024 GNU GPL V3.0\nPCB Rev. 1.2"
+	(gr_text "ESP32 fencing scoring device / weapons tester\ngithub.com/pietwauters/esp32_scoring_device_hardware\n©Piet Wauters 2024 GNU GPL V3.0\nPCB Rev. 1.2b"
 		(at 139.78 86.04 0)
 		(layer "B.SilkS")
@@
 		)
 	)
-	(gr_text "Fencing 3 weapons\n█ scoring device\n█ tester\nPCB Rev. 1.2\n"
+	(gr_text "Fencing 3 weapons\n█ scoring device\n█ tester\nPCB Rev. 1.2b\n"
 		(at 127.762 89.408 0)
 		(layer "F.SilkS")
